File: powerTimerPCB/powerTimer.kicad_pcb (KiCad board)
At the start: 2 copper layers, 35.4 x 25.6 mm, 34 parts, among them J1 Conn_01x02, J2 Conn_01x06, Q1 AO3401A, Q2 S8050H, Q3 S8050H, Q4 AO3401A, Q5 AO3401A, SW1 TS-1185EC-C-D-B, U1 RV-3028-C7 32.768KHZ 1PPM TA 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

Commit message: Minor change on MOSFET Q5 polarity
Parts:
- removed R12, R13: 0, Resistor_SMD:R_0603_1608Metric_Pad0.98x0.95mm_HandSolder
- added R14: 10K, Resistor_SMD:R_0603_1608Metric_Pad0.98x0.95mm_HandSolder, F.Cu at (125.3, 92.8)
Connections:
- Q5 pad 2: Net-(D1-A) -> +3.3V
- Q5 pad 3: +3.3V -> Net-(D1-A)
- R10 pad 1: Net-(R10-Pad1) -> +VPMU3.3
- R11 pad 1: Net-(R10-Pad1) -> +VPMU3.3
- U1 pad 6: GND -> Net-(U1-VBACKUP)
Routing:
- net Net-(U1-VBACKUP): track 0.00 -> 17.7 mm, vias 0 -> 2
- net Net-(R10-Pad1): track 11.6 -> 0.00 mm, vias 2 -> 0
- net GND: track 20.3 -> 31.7 mm, vias 1 -> 2
- net +3.3V: track 28.8 -> 32.3 mm, vias 10 -> 9
- net +VPMU3.3: track 32.2 -> 30.3 mm
- net Net-(D1-A): track 12.8 -> 14.3 mm
Other:
- board text added: "powerTimer-devOnChip"
- board text removed: "powerTimer"
