File: powerTimerPCB/powerTimer.kicad_sch (KiCad schematic)
At the start: 33 parts, among them J1 Conn_01x02, J2 Conn_01x06, Q1 AO3401A, Q2 S8050H, Q3 S8050H, Q4 AO3401A, Q5 AO3401A, SW1 TS-1185EC-C-D-B, U1 RV-3028-C7 32.768KHZ 1PPM TA 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

Commit message: Minor change on MOSFET Q5 polarity
Parts:
- removed R12, R13: 0, Resistor_SMD:R_0603_1608Metric_Pad0.98x0.95mm_HandSolder, symbol Device:R
- added R14: 10K, Resistor_SMD:R_0603_1608Metric_Pad0.98x0.95mm_HandSolder, symbol Device:R
Connections:
- net +3.3V: now also Q5.2 (S); no longer Q5.3 (D)
- net +VPMU3.3: now also R10.1, R11.1
- net GND: now also R14.2; no longer U1.6 (VBACKUP)
- net at D1.2 (A): now also Q5.3 (D); no longer Q5.2 (S)
- new net: R14.1, U1.6 (VBACKUP)
Other:
- note removed: "NC (Pull-Up same level as output)"
- moved on the sheet: Q5
